Commit message: updatec model to make a second link  and base link 0 length

File: arm.urdf (robot description, URDF)
Before this commit: robot 3dof_thrower, 4 links, 3 joints
Links:
- added link link_3; visual capsule length=0.2 radius=0.035
- link link_1: geometry visual capsule length=0.0 radius=0.05
Joints:
- added joint joint_4: type fixed, parent link_3, child cup_link, origin xyz=0 0 0.2
- joint joint_2: origin xyz=0 0 0.5 -> xyz=0 0 0.0
- joint joint_3: child cup_link -> link_3

Commit message: adding training script with config and wandb integration

File: arm.urdf (robot description, URDF)
Before this commit: robot 3dof_thrower, 5 links, 4 joints
Links:
- link base_link: mass None -> 5.0; geometry collision cylinder length=0.1 radius=0.2; visual cylinder length=0.1 radius=0.2
- link cup_link: mass None -> 0.2
- link link_1: mass None -> 0.6; geometry collision capsule length=0.1 radius=0.05; visual capsule length=0.1 radius=0.05
- link link_2: mass None -> 0.8; geometry collision capsule length=0.5 radius=0.04; visual capsule length=0.5 radius=0.04
- link link_3: mass None -> 0.4; geometry collision capsule length=0.2 radius=0.035; visual capsule length=0.2 radius=0.035
Joints:
- joint joint_1: origin xyz=0 0 0.05 -> xyz=0 0 0.05 rpy=0 0 0
- joint joint_2: origin xyz=0 0 0.0 -> xyz=0 0 0.1 rpy=0 0 0
- joint joint_3: origin xyz=0 0 0.5 -> xyz=0 0 0.5 rpy=0 0 0
- joint joint_4: origin xyz=0 0 0.2 -> xyz=0 0 0.2 rpy=0 0 0
